File: Glove.kicad_pcb (KiCad board)
At the start: 4 copper layers, 46 x 29.5 mm, 53 parts, among them J1 USB_C_Receptacle_USB2.0_14P, J2 Conn_01x08, J3 Conn_01x02_Socket, SW2 SW_SPDT, SW3 TS-1187A-B-A-B, U1 ESP32-C3-WROOM-02, U2 XC6220B331MR, U3 PCA9546APW,118, U5 DRV2605YZFR, U6 DRV2605YZFR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

Commit message: Added button connector
Parts:
- added J4: Conn_01x02, Connector_PinHeader_2.54mm:PinHeader_1x02_P2.54mm_Vertical, F.Cu at (81.7, 127.2)
- added JP4: SolderJumper_2_Open, Jumper:SolderJumper-2_P1.3mm_Open_RoundedPad1.0x1.5mm, F.Cu at (58.1, 124.4)
- added JP5: SolderJumper_2_Open, Jumper:SolderJumper-2_P1.3mm_Open_RoundedPad1.0x1.5mm, F.Cu at (55.9, 127.5)
- added JP6: SolderJumper_2_Open, Jumper:SolderJumper-2_P1.3mm_Open_RoundedPad1.0x1.5mm, F.Cu at (58.5, 127.5)
- moved R1 12.6 mm to (68.5, 128.1)
- moved R2 12.6 mm to (67.5, 128.1)
- moved D6 11.6 mm to (88.9, 116.4), turned to -90 degrees
- moved R16 5.82 mm to (78.7, 120.9)
Connections:
- U1 pad 11: unconnected-(U1-IO20/RXD-Pad11) -> Net-(J4-Pin_1)
- U1 pad 4: unconnected-(U1-IO5-Pad4) -> Net-(JP5-A)
- U1 pad 5: unconnected-(U1-IO6-Pad5) -> Net-(JP4-A)
- U1 pad 6: unconnected-(U1-IO7-Pad6) -> Net-(JP6-A)
Routing:
- net Net-(JP6-A): track 0.00 -> 19.4 mm, vias 0 -> 2
- net Net-(JP5-A): track 0.00 -> 18.9 mm
- net Net-(JP4-A): track 0.00 -> 13.8 mm
- net Net-(J4-Pin_1): track 0.00 -> 11.3 mm, vias 0 -> 1
- net Net-(D6-A): track 4.02 -> 11.9 mm
- net Net-(U1-IO21/TXD): track 12.2 -> 5.92 mm
- net Net-(JP1-B): track 3.07 -> 6.16 mm, vias 0 -> 2
- net GND: track 56.4 -> 58.5 mm, vias 102 -> 96
- net /CC2: track 10.4 -> 12.0 mm
- net Net-(J3-Pin_2): track 14.0 -> 15.5 mm, vias 0 -> 1
- net /CC1: track 11.8 -> 10.6 mm
Other:
- board text added: "J1"
- board text added: "J2"
- board text added: "J3"
- board text removed: "⎓ 3.0-4.2V"
